Commit message: using kobuki model that runs ok, still not smooth enough while heading straight.

File: kobuki_description/urdf/kobuki.urdf.xacro (robot description, xacro)
@@ -7,8 +7,8 @@
  -->
 <robot name="kobuki" xmlns:xacro="http://ros.org/wiki/xacro">
-  <xacro:include filename="$(find kobuki_description)/urdf/common_properties.urdf.xacro"/>
-  <xacro:include filename="$(find kobuki_description)/urdf/kobuki_gazebo.urdf.xacro"/>
+  <xacro:include filename="$(find MSTC_Star_update)/kobuki_description/urdf/common_properties.urdf.xacro"/>
+  <xacro:include filename="$(find MSTC_Star_update)/kobuki_description/urdf/kobuki_gazebo.urdf.xacro"/>
   <!-- Kobuki -->
-  <xacro:macro name="kobuki">
+  <!-- <xacro:macro name="kobuki"> -->
     <link name="base_footprint"/>
     <!--
@@ -30,5 +30,5 @@
         <geometry>
           <!-- new mesh -->
-          <mesh filename="package://kobuki_description/meshes/main_body.dae" />
+          <mesh filename="package://MSTC_Star_update/kobuki_description/meshes/main_body.dae" />
         </geometry>
         <origin xyz="0.001 0 0.05199" rpy="0 0 0"/>
@@ -65,5 +65,5 @@
       <visual>
         <geometry>
-          <mesh filename="package://kobuki_description/meshes/wheel.dae"/>
+          <mesh filename="package://MSTC_Star_update/kobuki_description/meshes/wheel.dae"/>
         </geometry>
         <origin xyz="0 0 0" rpy="0 0 0"/>
@@ -92,5 +92,5 @@
       <visual>
         <geometry>
-          <mesh filename="package://kobuki_description/meshes/wheel.dae"/>
+          <mesh filename="package://MSTC_Star_update/kobuki_description/meshes/wheel.dae"/>
         </geometry>
         <origin xyz="0 0 0" rpy="0 0 0"/>
@@ -210,4 +210,4 @@
     <!-- Kobuki Gazebo simulation details -->
     <kobuki_sim/>
-  </xacro:macro>
+  <!-- </xacro:macro> -->
 </robot>

File: kobuki_description/urdf/kobuki_gazebo.urdf.xacro (robot description, xacro)
@@ -1,5 +1,5 @@
 <?xml version="1.0"?>
 <robot name="kobuki_sim" xmlns:xacro="http://ros.org/wiki/xacro">
-  <xacro:macro name="kobuki_sim">
+  <!-- <xacro:macro name="kobuki_sim"> -->
 	  <gazebo reference="wheel_left_link">
 	    <mu1>1.0</mu1>
@@ -160,5 +160,5 @@
       </sensor>
 	  </gazebo>
-	  <gazebo>
+	  <!-- <gazebo>
 	    <plugin name="kobuki_controller" filename="libgazebo_ros_kobuki.so">
 	      <publish_tf>1</publish_tf>
@@ -176,5 +176,39 @@
         <imu_name>imu</imu_name>
 	    </plugin>
-	  </gazebo>
-  </xacro:macro>
+	  </gazebo> -->
+	<gazebo>
+      <plugin name="kobuki_controller" filename="libgazebo_ros_diff_drive.so">
+		<commandTopic>cmd_vel</commandTopic>
+		<odometryTopic>odom</odometryTopic>
+		<odometryFrame>odom</odometryFrame>
+		<odometrySource>world</odometrySource>
+		<publishOdomTF>false</publishOdomTF>
+		<robotBaseFrame>base_footprint</robotBaseFrame>
+		<publishWheelTF>true</publishWheelTF>
+		<publishTf>true</publishTf>
+		<publishWheelJointState>true</publishWheelJointState>
+		<legacyMode>false</legacyMode>
+		<updateRate>30</updateRate>
+		<leftJoint>wheel_left_joint</leftJoint>
+		<rightJoint>wheel_right_joint</rightJoint>
+		<wheelSeparation>0.230</wheelSeparation>
+		<wheelDiameter>0.07</wheelDiameter>
+		<wheelAcceleration>1</wheelAcceleration>
+		<wheelTorque>5</wheelTorque>
+		<rosDebugLevel>na</rosDebugLevel>
+      </plugin>
+    </gazebo>
+	<gazebo>
+	  <plugin name="p3d_base_controller" filename="libgazebo_ros_p3d.so">
+		<alwaysOn>true</alwaysOn>
+		<updateRate>50</updateRate>
+		<bodyName>base_footprint</bodyName>
+		<topicName>ground_truth/state</topicName>
+		<gaussianNoise>0.01</gaussianNoise>
+		<frameName>map</frameName>
+		<xyzOffsets>0 0 0</xyzOffsets>
+		<rpyOffsets>0 0 0</rpyOffsets>
+	  </plugin>
+    </gazebo>
+  <!-- </xacro:macro> -->
 </robot>

File: kobuki_description/urdf/kobuki_standalone.urdf.xacro (robot description, xacro)
@@ -6,5 +6,5 @@
        xmlns:xacro="http://ros.org/wiki/xacro">
   <!-- Defines the kobuki component tag. -->
-  <xacro:include filename="$(find kobuki_description)/urdf/kobuki.urdf.xacro" />
+  <xacro:include filename="$(find MSTC_Star_update)/kobuki_description/urdf/kobuki.urdf.xacro" />
   <kobuki/>
 </robot>

Commit message: steady version of TMSTC* with teb local planner

File: kobuki_description/urdf/kobuki.urdf.xacro (robot description, xacro)
@@ -167,5 +167,5 @@
     </link>
     <joint name="cliff_sensor_left_joint" type="fixed">
-      <origin xyz="0.08734 0.13601 0.0214" rpy="0 ${M_PI/2} 0" />
+      <origin xyz="0 -0.1 0.05" rpy="0 0 -1.5708" />
       <parent link="base_link"/>
       <child link="cliff_sensor_left_link" />
@@ -181,5 +181,5 @@
     </link>
     <joint name="cliff_sensor_right_joint" type="fixed">
-      <origin xyz="0.085 -0.13601 0.0214" rpy="0 ${M_PI/2} 0" />
+      <origin xyz="0 0.1 0.05" rpy="0 0 0" />
       <parent link="base_link"/>
       <child link="cliff_sensor_right_link" />
@@ -195,5 +195,5 @@
     </link>
     <joint name="cliff_sensor_front_joint" type="fixed">
-      <origin xyz="0.156 0.00 0.0214" rpy="0 ${M_PI/2} 0" />
+      <origin xyz="0 0.00 0.05" rpy="0 0 -${M_PI/2}" />
       <parent link="base_link"/>
       <child link="cliff_sensor_front_link" />

File: kobuki_description/urdf/kobuki_gazebo.urdf.xacro (robot description, xacro)
@@ -108,30 +108,31 @@
 	  <gazebo reference="cliff_sensor_front_link">
 	    <sensor type="ray" name="cliff_sensor_front">
-	      <always_on>true</always_on>
-	      <update_rate>50</update_rate>
-	      <visualize>true</visualize>
-	      <ray>
-	        <scan>
-	          <horizontal>
-	            <samples>50</samples>
-	            <resolution>1.0</resolution>
-	            <min_angle>-0.0436</min_angle>  <!-- -2.5 degree -->
-	            <max_angle>0.0436</max_angle> <!-- 2.5 degree -->
-	          </horizontal>
-<!-- 	          Can't use vertical rays until this bug is resolved: -->
-<!--            https://bitbucket.org/osrf/gazebo/issue/509/vertical-sensor-doesnt-works -->
-<!-- 	          <vertical> -->
-<!-- 	            <samples>50</samples> -->
-<!-- 	            <resolution>1.0</resolution> -->
-<!-- 	            <min_angle>-0.0436</min_angle>  -2.5 degree -->
-<!-- 	            <max_angle>0.0436</max_angle> 2.5 degree -->
-<!-- 	          </vertical> -->
-	        </scan>
-	        <range>
-	          <min>0.01</min>
-	          <max>0.15</max>
-	          <resolution>1.0</resolution>
-	        </range>
-	      </ray>
+			<!-- <pose>0 0 0 0 0 0</pose> -->
+			<visualize>true</visualize>
+			<update_rate>10</update_rate>
+			<ray>
+				<scan>
+				<horizontal>
+					<samples>360</samples>
+					<resolution>1</resolution>
+					<min_angle>0</min_angle>
+					<max_angle>3.14159</max_angle>
+				</horizontal>
+				</scan>
+				<range>
+					<min>0.20</min>
+					<max>4</max>
+					<resolution>0.015</resolution>
+				</range>
+				<noise>
+				<type>gaussian</type>
+				<mean>0.0</mean>
+				<stddev>0.01</stddev>
+				</noise>
+			</ray>
+			<plugin name="gazebo_ros_lds_lfcd_controller" filename="libgazebo_ros_laser.so">
+				<topicName>laser/scan</topicName>
+				<frameName>cliff_sensor_front_link</frameName>
+			</plugin>
 	    </sensor>
 	  </gazebo>
